File: hardware/paracaidas-matrice400/paracaidas-matrice400.kicad_sch (KiCad schematic)
At the start: 0 parts

Commit message: Implementa esquemático KiCad completo: sistema paracaídas DJI Matrice 400
- 31 componentes: PIC18LF25K22, MPU-6050, MT3608, MCP1700-3302E,
  IRLZ44N, 2N3904, 1N4007, resistencias, capacitores, inductor,
  LEDs, buzzer, solenoid, batería, switches, conectores UART/ICSP
- 24 nets verificados con kicad-happy: SCL/SDA/I2C, MPU_INT,
  SOL_CTRL, BUZ_CTRL, LED1/LED2, MCLR, UART_TX/RX, PGC/PGD,
  VBAT, VBAT_SW, BOOST_SW, BOOST_FB, +3V3, +5V, GND, DRAIN_Q1
- gen_sch.py: generador Python que aplica la misma fórmula de
  coordenadas que el analizador (abs_y = cy - rpy, Y invertido)

Co-Authored-By: Claude Sonnet 4.6 <noreply@anthropic.com>
Parts:
- added BT1: LiPo_1S_1000mAh, symbol Device:Battery_Cell
- added BZ1: Buzzer_5V, symbol Device:Buzzer
- added C1, C3, C5: 100nF, symbol Device:C
- added C2: 10uF, symbol Device:C
- added C4: 100uF, symbol Device:C
- added D1: 1N4007, symbol Device:D
- added J1: UART_Debug, symbol Connector_Generic:Conn_01x04
- added J2: ICSP_PICKit, symbol Connector_Generic:Conn_01x04
- added L1: 22uH_1A, symbol Device:L
- added LED1: LED_Verde, symbol Device:LED
- added LED2: LED_Rojo, symbol Device:LED
- added Q1: IRLZ44N, symbol Device:Q_NMOS_GDS
- added Q2: 2N3904, symbol Device:Q_NPN_BCE
- added R1, R2: 10k, symbol Device:R
- added R3, R4: 330, symbol Device:R
- added R5, R6: 4k7, symbol Device:R
- added R7: 1k, symbol Device:R
- added R_FB1: 750k, symbol Device:R
- added R_FB2: 100k, symbol Device:R
- added SOL1: Solenoid_5V, symbol Mechanical:Solenoid
- added SW1: SW_ON-OFF, symbol Switch:SW_SPST
- added SW2: SW_Push_MCLR, symbol Switch:SW_Push
- added U1: PIC18LF25K22, symbol MCU:PIC18LF25K22
- added U2: MPU-6050, symbol Sensor_Motion:MPU-6050
- added U3: MCP1700-3302E, symbol Regulator_Linear:MCP1700-3302E
- added U4: MT3608, symbol Regulator_Switching:MT3608
Connections:
- new net +3V3: C1.1 (+), C2.1 (+), C3.1 (+), R1.1, R5.1, R6.1, U1.20 (VDD), U2.1 (VCC), U3.3 (OUT)
- new net +5V: BZ1.+, C4.1 (+), D1.K, J1.4 (Pin_4), J2.1 (Pin_1), L1.2, R_FB1.1, SOL1.1, U4.6 (BS)
- new net BOOST_FB: R_FB1.2, R_FB2.1, U4.3 (FB)
- new net BOOST_SW: L1.1, U4.5 (SW)
- new net BUZ_CTRL: R7.2, U1.11 (RC0)
- new net BZ_COL: BZ1.K, Q2.C
- new net DRAIN_Q1: D1.A, Q1.D, SOL1.2
- new net GND: BT1.-, C1.2 (-), C2.2 (-), C3.2 (-), C4.2 (-), C5.2 (-), J1.1 (Pin_1), J2.2 (Pin_2), LED1.K, LED2.K, Q1.S, Q2.E, R2.2, R_FB2.2, SW2.2 (B), U1.19 (VSS), U1.8 (VSS), U2.2 (GND), U2.6 (AD0), U3.2 (GND), U4.2 (GND)
- new net LED1_A: LED1.A, R3.1
- new net LED1_CTRL: R3.2, U1.2 (RA0)
- new net LED2_A: LED2.A, R4.1
- new net LED2_CTRL: R4.2, U1.3 (RA1)
- new net MCLR: R1.2, SW2.1 (A), U1.1 (MCLR)
- new net MPU_INT: U1.21 (RB0), U2.5 (INT)
- new net PGC: J2.3 (Pin_3), U1.27 (RB6)
- new net PGD: J2.4 (Pin_4), U1.28 (RB7)
- new net Q2_BASE: Q2.B, R7.1
- new net SCL: R5.2, U1.14 (RC3), U2.3 (SCL)
- new net SDA: R6.2, U1.15 (RC4), U2.4 (SDA)
- new net SOL_CTRL: Q1.G, R2.1, U1.13 (RC2)
- new net UART_RX: J1.2 (Pin_2), U1.18 (RC7)
- new net UART_TX: J1.3 (Pin_3), U1.17 (RC6)
- new net VBAT: BT1.+, SW1.1 (A)
- new net VBAT_SW: C5.1 (+), SW1.2 (B), U3.1 (IN), U4.1 (IN), U4.4 (EN)
- no-connect marks 0 -> 15
