File: hardware/paracaidas-matrice400/paracaidas-matrice400.kicad_sch (KiCad schematic)
At the start: 31 parts, among them J1 UART_Debug, J2 ICSP_PICKit, Q1 IRLZ44N, Q2 2N3904, SW1 SW_ON-OFF, SW2 SW_Push_MCLR, U1 PIC18LF25K22, U2 MPU-6050, U3 MCP1700-3302E, U4 MT3608

Commit message: Refactor code structure for improved readability and maintainability
Parts:
- BT1, SOL1: footprint (none) -> Connector_PinHeader_2.54mm:PinHeader_1x02_P2.54mm_Vertical
- BZ1: footprint (none) -> Buzzer_Beeper:ABT-410-RC
- C1, C3, C5: footprint (none) -> Capacitor_THT:C_Disc_D5.0mm_W2.5mm_P5.00mm
- C2, C4: footprint (none) -> Capacitor_THT:CP_Radial_D6.3mm_P2.50mm
- D1: footprint (none) -> Diode_THT:D_DO-41_SOD81_P10.16mm_Horizontal
- J1, J2: footprint (none) -> Connector_PinHeader_2.54mm:PinHeader_1x04_P2.54mm_Vertical
- L1: footprint (none) -> Inductor_THT:L_Axial_L5.3mm_D2.2mm_P10.16mm_Horizontal
- LED1, LED2: footprint (none) -> LED_THT:LED_D5.0mm
- Q1: footprint (none) -> Package_TO_SOT_THT:TO-220-3_Vertical
- Q2: footprint (none) -> Package_TO_SOT_THT:TO-92_Inline
- R1, R2, R3, R4, R5, R6, R7, R_FB1, R_FB2: footprint (none) -> Resistor_THT:R_Axial_DIN0207_L6.3mm_D2.5mm_P10.16mm_Horizontal
- SW1: footprint (none) -> Button_Switch_THT:SW_Slide_1P2T_CK_OS102011MS2Q
- SW2: footprint (none) -> Button_Switch_THT:SW_PUSH_6mm
- U1: footprint (none) -> Package_DIP:DIP-28_W7.62mm
- U2: footprint (none) -> Connector_PinHeader_2.54mm:PinHeader_2x04_P2.54mm_Vertical
- U3: footprint (none) -> Package_TO_SOT_SMD:SOT-23
- U4: footprint (none) -> Package_TO_SOT_SMD:SOT-23-6

Commit message: Add lock file for paracaidas-matrice400 schematic with user and hostname information
Parts:
- removed BT1: LiPo_1S_1000mAh, Connector_PinHeader_2.54mm:PinHeader_1x02_P2.54mm_Vertical, symbol Device:Battery_Cell
- removed BZ1: Buzzer_5V, Buzzer_Beeper:ABT-410-RC, symbol Device:Buzzer
- removed C1, C3, C5: 100nF, Capacitor_THT:C_Disc_D5.0mm_W2.5mm_P5.00mm, symbol Device:C
- removed C2: 10uF, Capacitor_THT:CP_Radial_D6.3mm_P2.50mm, symbol Device:C
- removed C4: 100uF, Capacitor_THT:CP_Radial_D6.3mm_P2.50mm, symbol Device:C
- removed D1: 1N4007, Diode_THT:D_DO-41_SOD81_P10.16mm_Horizontal, symbol Device:D
- removed J1: UART_Debug, Connector_PinHeader_2.54mm:PinHeader_1x04_P2.54mm_Vertical, symbol Connector_Generic:Conn_01x04
- removed J2: ICSP_PICKit, Connector_PinHeader_2.54mm:PinHeader_1x04_P2.54mm_Vertical, symbol Connector_Generic:Conn_01x04
- removed L1: 22uH_1A, Inductor_THT:L_Axial_L5.3mm_D2.2mm_P10.16mm_Horizontal, symbol Device:L
- removed LED1: LED_Verde, LED_THT:LED_D5.0mm, symbol Device:LED
- removed LED2: LED_Rojo, LED_THT:LED_D5.0mm, symbol Device:LED
- removed Q1: IRLZ44N, Package_TO_SOT_THT:TO-220-3_Vertical, symbol Device:Q_NMOS_GDS
- removed Q2: 2N3904, Package_TO_SOT_THT:TO-92_Inline, symbol Device:Q_NPN_BCE
- removed R1, R2: 10k, Resistor_THT:R_Axial_DIN0207_L6.3mm_D2.5mm_P10.16mm_Horizontal, symbol Device:R
- removed R3, R4: 330, Resistor_THT:R_Axial_DIN0207_L6.3mm_D2.5mm_P10.16mm_Horizontal, symbol Device:R
- removed R5, R6: 4k7, Resistor_THT:R_Axial_DIN0207_L6.3mm_D2.5mm_P10.16mm_Horizontal, symbol Device:R
- removed R7: 1k, Resistor_THT:R_Axial_DIN0207_L6.3mm_D2.5mm_P10.16mm_Horizontal, symbol Device:R
- removed R_FB1: 750k, Resistor_THT:R_Axial_DIN0207_L6.3mm_D2.5mm_P10.16mm_Horizontal, symbol Device:R
- removed R_FB2: 100k, Resistor_THT:R_Axial_DIN0207_L6.3mm_D2.5mm_P10.16mm_Horizontal, symbol Device:R
- removed SOL1: Solenoid_5V, Connector_PinHeader_2.54mm:PinHeader_1x02_P2.54mm_Vertical, symbol Mechanical:Solenoid
- removed SW1: SW_ON-OFF, Button_Switch_THT:SW_Slide_1P2T_CK_OS102011MS2Q, symbol Switch:SW_SPST
- removed SW2: SW_Push_MCLR, Button_Switch_THT:SW_PUSH_6mm, symbol Switch:SW_Push
- removed U1: PIC18LF25K22, Package_DIP:DIP-28_W7.62mm, symbol MCU:PIC18LF25K22
- removed U2: MPU-6050, Connector_PinHeader_2.54mm:PinHeader_2x04_P2.54mm_Vertical, symbol Sensor_Motion:MPU-6050
- removed U3: MCP1700-3302E, Package_TO_SOT_SMD:SOT-23, symbol Regulator_Linear:MCP1700-3302E
- removed U4: MT3608, Package_TO_SOT_SMD:SOT-23-6, symbol Regulator_Switching:MT3608
Connections:
- no-connect marks 15 -> 0
